File: fm1-midi-dongle.kicad_pcb (KiCad board)
At the start: 4 copper layers, 20 x 37.7 mm, 29 parts, among them J1 911-321B2028S10100, J2 TYPE-C-31-M-12, J3 PJ-320D, J4 PJ-320D, U1 CH32X035G8U6, U2 XC6206P332MR, U3 SY6280AAC, U4 H11L1SM, U5 SN74LVC1G3157

Commit message: v6.1: case screw holes, milled aluminium + printed + sheet-metal cases
- board: two M1.6 case holes (H1 between the jacks, H2 beside the USB-A), board-only NPTH;
  silk keeps text off the case bosses; DRC back to the v6 baseline
- case/gen_case.py: one design, CASE=alu (CNC 6061) or CASE=print. Split at the jacks' axis so
  every port is half in each half (the v6 snap case split at the board face could not close
  without the jack-end wall bending ~2 mm). 2 x M1.6 x 6 countersunk screws through the board.
  Pockets hug the parts and are shaped for the cutter radius.
- case/gen_case_sheet.py: 0.8 mm 5052 two-U box (base: bottom + sides, cover: top + ends with
  M2 clinch-nut tabs), connectors 0.9 mm behind the walls
- check_fit.py: fit, straight-down assembly sweep, screws / hardware: 0 collisions for all three

Co-Authored-By: Claude Opus 5.5 <noreply@anthropic.com>
Claude-Session: https://claude.ai/code/session_01Dtfv3zuhZTs975LiSXznFQ
Parts:
- added H1: M1.6 hole, fm1_dongle:MountingHole_1.7mm_NPTH, F.Cu at (0.00, 34.4)
- added H2: M1.6 hole, fm1_dongle:MountingHole_1.7mm_NPTH, F.Cu at (8.30, 3.00)
